Commit message: Edit code

File: code/lecture5/simple_robot.urdf (robot description, URDF)
Before this commit: robot simple_robot, 3 links, 2 joints
Joints:
- removed joint base_to_left_arm_joint
- removed joint base_to_right_arm_joint
- added joint base_to_left_arm: type fixed, parent base_link, child left_arm, origin xyz=-0.2 0.01 0 rpy=0 0 0
- added joint base_to_right_arm: type fixed, parent base_link, child right_arm, origin xyz=0.2 0.01 0 rpy=0 0 0
